Commit message: after course

File: src/gazebo_env/model/humanoid.urdf (robot description, URDF)
Before this commit: robot human, 19 links, 18 joints
Links:
- link chest: geometry collision box size=0.1125 0.0975 0.14; collision cylinder length=0.1146 radius=0.008
- link head: geometry collision sphere radius=0.0284086; collision sphere radius=0.0305397
- link left_arm: geometry collision box size=0.1271 0.048 0.028; visual mesh filename=meshes/left_arm.STL
- link left_foot: geometry collision box size=0.0659544 0.149954 0.012; collision box size=0.087 0.147 0.006
- link left_hand: geometry collision box size=0.120244 0.027 0.003; collision cylinder length=0.003 radius=0.02
- link left_leg_ankle: geometry collision box size=0.003 0.029 0.0651; collision box size=0.0035 0.029 0.0651
- link left_leg_knee: geometry collision cylinder length=0.0055 radius=0.014; collision cylinder length=0.0055 radius=0.014
- link left_leg_pitch: geometry collision box size=0.0539 0.0402 0.0015; collision box size=0.0539 0.0402 0.0015
- link left_leg_roll: geometry collision box size=0.028997 0.0035 0.0553928; collision box size=0.0403884 0.038 0.0611006
- link left_leg_yaw: geometry collision box size=0.041 0.0637 0.003; visual mesh filename=meshes/left_leg_yaw.STL
- link neck: geometry collision box size=0.0302 0.0356 0.0396; collision box size=0.0342 0.0355 0.015
- link right_arm: geometry collision box size=0.1271 0.048 0.028; visual mesh filename=meshes/right_arm.STL
- link right_foot: geometry collision box size=0.0659544 0.149954 0.012; collision box size=0.087 0.147 0.006
- link right_hand: geometry collision box size=0.120244 0.027 0.003; collision cylinder length=0.003 radius=0.02
- link right_leg_ankle: geometry collision box size=0.003 0.029 0.0651; collision box size=0.0035 0.029 0.0651
- link right_leg_knee: geometry collision cylinder length=0.0055 radius=0.014; collision cylinder length=0.0055 radius=0.014
- link right_leg_pitch: geometry collision box size=0.0539 0.0402 0.0015; collision box size=0.0539 0.0402 0.0015
- link right_leg_roll: geometry collision box size=0.028997 0.0035 0.0553928; collision box size=0.0403884 0.038 0.0611006
- link right_leg_yaw: geometry collision box size=0.041 0.0637 0.003; visual mesh filename=meshes/right_leg_yaw.STL
